Commit message: update README, cleanup robot urdf

File: waiteronix/urdf/waiteronix.xacro (robot description, xacro)
@@ -1,10 +1,9 @@
-<?xml version="1.0" encoding="utf-8"?>
-<!-- This URDF was automatically created by SolidWorks to URDF Exporter! Originally created by Stephen Brawner (brawner@gmail.com)
+<?xml version="1.0" ?>
+<robot name="waiteronix" xmlns:xacro="http://www.ros.org/wiki/xacro">
+  <!-- This URDF was automatically created by SolidWorks to URDF Exporter! Originally created by Stephen Brawner (brawner@gmail.com)
      Commit Version: 1.6.0-4-g7f85cfe  Build Version: 1.6.7995.38578
      For more information, please see http://wiki.ros.org/sw_urdf_exporter -->
-<robot
-  name="waiteronix">
-  <link name="dummy">
-   </link>
+  <link name="robot_footprint">
+  </link>
   <link
     name="base_link">
@@ -48,5 +47,5 @@
   </link>
   <joint name="dummy_joint" type="fixed">
-    <parent link="dummy"/>
+    <parent link="robot_footprint"/>
     <child link="base_link"/>
    </joint>
@@ -269,46 +268,4 @@
       xyz="1 0 0" />
   </joint>
-   <!--camera plugin-->
-  <gazebo reference="Camera">
-  <sensor name="Camera_camera" type="depth">
-    <update_rate>20</update_rate>
-    <camera>
-      <horizontal_fov>1.047198</horizontal_fov>
-      <image>
-        <width>640</width>
-        <height>480</height>
-        <format>R8G8B8</format>
-      </image>
-      <clip>
-        <near>0.05</near>
-        <far>3</far>
-      </clip>
-    </camera>
-    <plugin name="Camera_controller" filename="libgazebo_ros_openni_kinect.so">
-      <baseline>0.2</baseline>
-      <alwaysOn>true</alwaysOn>
-      <updateRate>1.0</updateRate>
-      <cameraName>kinect_ir</cameraName>
-      <imageTopicName>/kinect/color/image_raw</imageTopicName>
-      <cameraInfoTopicName>/kinect/color/camera_info</cameraInfoTopicName>
-      <depthImageTopicName>/kinect/depth/image_raw</depthImageTopicName>
-      <depthImageInfoTopicName>/kinect/depth/camera_info</depthImageInfoTopicName>
-      <pointCloudTopicName>/kinect/depth/points</pointCloudTopicName>
-      <frameName>Camera</frameName>
-      <pointCloudCutoff>0.5</pointCloudCutoff>
-      <pointCloudCutoffMax>3.0</pointCloudCutoffMax>
-      <distortionK1>0.00000001</distortionK1>
-      <distortionK2>0.00000001</distortionK2>
-      <distortionK3>0.00000001</distortionK3>
-      <distortionT1>0.00000001</distortionT1>
-      <distortionT2>0.00000001</distortionT2>
-      <CxPrime>0</CxPrime>
-      <Cx>0</Cx>
-      <Cy>0</Cy>
-      <focalLength>0</focalLength>
-      <hackBaseline>0</hackBaseline>
-    </plugin>
-  </sensor>
-</gazebo>
   <link
     name="Lidar">
@@ -364,40 +321,4 @@
       xyz="0 0 1" />
   </joint>
-    <!--rplidar a1 plugin-->
-    <gazebo reference="Lidar">
-        <sensor type="ray" name="head_hokuyo_sensor">
-            <pose>0 0 0 0 0 0</pose>
-            <visualize>true</visualize>
-            <update_rate>40</update_rate>
-            <ray>
-                <scan>
-                    <horizontal>
-                        <samples>360</samples>
-                        <resolution>1</resolution>
-                        <min_angle>-3.141592654</min_angle>
-                        <max_angle>3.141592654</max_angle>
-                    </horizontal>
-                </scan>
-                <range>
-                    <min>0.15</min>
-                    <max>6.0</max>
-                    <resolution>0.5</resolution>
-                </range>
-                <noise>
-                    <type>gaussian</type>
-                    <!-- Noise parameters based on published spec for Hokuyo laser
-                        achieving "+-30mm" accuracy at range < 10m.  A mean of 0.0m and
-                        stddev of 0.01m will put 99.7% of samples within 0.03m of the true
-                        reading. -->
-                    <mean>0.0</mean>
-                    <stddev>0.01</stddev>
-                </noise>
-            </ray>
-            <plugin name="gazebo_ros_head_hokuyo_controller" filename="libgazebo_ros_laser.so">
-                <topicName>/scan</topicName>
-                <frameName>Lidar</frameName>
-            </plugin>
-        </sensor>
-    </gazebo>
   <link
     name="IMU">
@@ -453,25 +374,4 @@
       xyz="0 0 1" />
   </joint>
-<!--imu plugin-->
-  <gazebo reference="IMU">
-    <gravity>true</gravity>
-    <sensor name="imu_sensor" type="imu">
-      <always_on>true</always_on>
-      <update_rate>100</update_rate>
-      <visualize>true</visualize>
-      <topic>__default_topic__</topic>
-      <plugin filename="libgazebo_ros_imu_sensor.so" name="imu_plugin">
-        <topicName>imu</topicName>
-        <bodyName>IMU</bodyName>
-        <updateRateHZ>10.0</updateRateHZ>
-        <gaussianNoise>0.0</gaussianNoise>
-        <xyzOffset>0 0 0</xyzOffset>
-        <rpyOffset>0 0 0</rpyOffset>
-        <frameName>IMU</frameName>
-        <initialOrientationAsReference>false</initialOrientationAsReference>
-      </plugin>
-      <pose>0 0 0 0 0 0</pose>
-    </sensor>
-  </gazebo>
   <link
     name="F_W_Front_Left">

Commit message: partioning the whole xacro  file into 4 files and modifying differential wheels parameters

File: waiteronix/urdf/waiteronix.xacro (robot description, xacro)
@@ -5,4 +5,7 @@
      For more information, please see http://wiki.ros.org/sw_urdf_exporter -->
   <xacro:include filename="$(find waiteronix)/urdf/waiteronix.gazebo"/>
+  <xacro:include filename="$(find waiteronix)/urdf/caster_wheels.xacro"/>
+  <xacro:include filename="$(find waiteronix)/urdf/diff_wheels.xacro"/>
+  <xacro:include filename="$(find waiteronix)/urdf/sensors.xacro"/>
   <link name="robot_footprint">
   </link>
@@ -104,486 +107,3 @@
       xyz="0 0 0" />
   </joint>
-  <link
-    name="Right_Wheel">
-    <inertial>
-      <origin
-        xyz="2.5996E-07 0.037854 6.57E-06"
-        rpy="0 0 0" />
-      <mass
-        value="1.21" />
-      <inertia
-        ixx="0.0022228"
-        ixy="-1.8762E-08"
-        ixz="1.5736E-09"
-        iyy="0.0036326"
-        iyz="-4.7418E-07"
-        izz="0.0022228" />
-    </inertial>
-    <visual>
-      <origin
-        xyz="0 0 0"
-        rpy="0 0 0" />
-      <geometry>
-        <mesh
-          filename="package://waiteronix/meshes/Right_Wheel.STL" />
-      </geometry>
-      <material
-        name="">
-        <color
-          rgba="0.75294 0.75294 0.75294 1" />
-      </material>
-    </visual>
-    <collision>
-      <origin
-        xyz="0 0 0"
-        rpy="0 0 0" />
-      <geometry>
-        <mesh
-          filename="package://waiteronix/meshes/Right_Wheel.STL" />
-      </geometry>
-    </collision>
-  </link>
-  <joint
-    name="Right_Wheel_Joint"
-    type="continuous">
-    <origin
-      xyz="-0.0087223 -0.224 0.054"
-      rpy="0 0 0" />
-    <parent
-      link="base_link" />
-    <child
-      link="Right_Wheel" />
-    <axis
-      xyz="0 -1 0" />
-    <limit
-      effort="40"
-      velocity="10" />
-  </joint>
-  <link
-    name="Left_Wheel">
-    <inertial>
-      <origin
-        xyz="2.5996E-07 -0.037854 6.57E-06"
-        rpy="0 0 0" />
-      <mass
-        value="1.21" />
-      <inertia
-        ixx="0.0022228"
-        ixy="1.8762E-08"
-        ixz="1.5736E-09"
-        iyy="0.0036326"
-        iyz="4.7418E-07"
-        izz="0.0022228" />
-    </inertial>
-    <visual>
-      <origin
-        xyz="0 0 0"
-        rpy="0 0 0" />
-      <geometry>
-        <mesh
-          filename="package://waiteronix/meshes/Left_Wheel.STL" />
-      </geometry>
-      <material
-        name="">
-        <color
-          rgba="0.75294 0.75294 0.75294 1" />
-      </material>
-    </visual>
-    <collision>
-      <origin
-        xyz="0 0 0"
-        rpy="0 0 0" />
-      <geometry>
-        <mesh
-          filename="package://waiteronix/meshes/Left_Wheel.STL" />
-      </geometry>
-    </collision>
-  </link>
-  <joint
-    name="Left_Wheel_Joint"
-    type="continuous">
-    <origin
-      xyz="-0.0087223 0.224 0.054"
-      rpy="0 0 0" />
-    <parent
-      link="base_link" />
-    <child
-      link="Left_Wheel" />
-    <axis
-      xyz="0 -1 0" />
-    <limit
-      effort="40"
-      velocity="10" />
-  </joint>
-  <link
-    name="Camera">
-    <inertial>
-      <origin
-        xyz="-0.027769 0.064365 -0.00028163"
-        rpy="0 0 0" />
-      <mass
-        value="0.55893" />
-      <inertia
-        ixx="0.0029329"
-        ixy="-9.3578E-07"
-        ixz="8.9611E-08"
-        iyy="0.00023177"
-        iyz="-9.4508E-09"
-        izz="0.0030272" />
-    </inertial>
-    <visual>
-      <origin
-        xyz="0 0 0"
-        rpy="0 0 0" />
-      <geometry>
-        <mesh
-          filename="package://waiteronix/meshes/Camera.STL" />
-      </geometry>
-      <material
-        name="">
-        <color
-          rgba="0.49412 0.49412 0.49412 1" />
-      </material>
-    </visual>
-    <collision>
-      <origin
-        xyz="0 0 0"
-        rpy="0 0 0" />
-      <geometry>
-        <mesh
-          filename="package://waiteronix/meshes/Camera.STL" />
-      </geometry>
-    </collision>
-  </link>
-  <joint
-    name="Camera_Joint"
-    type="fixed">
-    <origin
-      xyz="0.24478 -0.064307 0.0965"
-      rpy="0 0 0" />
-    <parent
-      link="base_link" />
-    <child
-      link="Camera" />
-    <axis
-      xyz="1 0 0" />
-  </joint>
-  <link
-    name="Lidar">
-    <inertial>
-      <origin
-        xyz="8.3267E-17 -1.9976E-15 -0.013917"
-        rpy="0 0 0" />
-      <mass
-        value="0.12331" />
-      <inertia
-        ixx="8.5672E-05"
-        ixy="-3.3087E-22"
-        ixz="-3.3193E-19"
-        iyy="8.5672E-05"
-        iyz="-1.4388E-23"
-        izz="0.00010203" />
-    </inertial>
-    <visual>
-      <origin
-        xyz="0 0 0"
-        rpy="0 0 0" />
-      <geometry>
-        <mesh
-          filename="package://waiteronix/meshes/Lidar.STL" />
-      </geometry>
-      <material
-        name="">
-        <color
-          rgba="0 0.75294 0 1" />
-      </material>
-    </visual>
-    <collision>
-      <origin
-        xyz="0 0 0"
-        rpy="0 0 0" />
-      <geometry>
-        <mesh
-          filename="package://waiteronix/meshes/Lidar.STL" />
-      </geometry>
-    </collision>
-  </link>
-  <joint
-    name="Lidar_Joint"
-    type="fixed">
-    <origin
-      xyz="0.185 0 0.21663"
-      rpy="0 0 0" />
-    <parent
-      link="base_link" />
-    <child
-      link="Lidar" />
-    <axis
-      xyz="0 0 1" />
-  </joint>
-  <link
-    name="IMU">
-    <inertial>
-      <origin
-        xyz="-1.8518E-16 -6.2326E-15 -0.005"
-        rpy="0 0 0" />
-      <mass
-        value="0.0007854" />
-      <inertia
-        ixx="1.1454E-08"
-        ixy="1.831E-25"
-        ixz="-3.3736E-23"
-        iyy="1.1454E-08"
-        iyz="1.7323E-23"
-        izz="9.8175E-09" />
-    </inertial>
-    <visual>
-      <origin
-        xyz="0 0 0"
-        rpy="0 0 0" />
-      <geometry>
-        <mesh
-          filename="package://waiteronix/meshes/IMU.STL" />
-      </geometry>
-      <material
-        name="">
-        <color
-          rgba="0 0.75294 0 1" />
-      </material>
-    </visual>
-    <collision>
-      <origin
-        xyz="0 0 0"
-        rpy="0 0 0" />
-      <geometry>
-        <mesh
-          filename="package://waiteronix/meshes/IMU.STL" />
-      </geometry>
-    </collision>
-  </link>
-  <joint
-    name="IMU_Joint"
-    type="fixed">
-    <origin
-      xyz="0 0 0.289"
-      rpy="0 0 0" />
-    <parent
-      link="base_link" />
-    <child
-      link="IMU" />
-    <axis
-      xyz="0 0 1" />
-  </joint>
-  <link
-    name="F_W_Front_Left">
-    <inertial>
-      <origin
-        xyz="0.13868 0.123 -1.4438E-14"
-        rpy="0 0 0" />
-      <mass
-        value="0.059636" />
-      <inertia
-        ixx="1.6012E-05"
-        ixy="-1.927E-20"
-        ixz="-9.0002E-22"
-        iyy="2.7287E-05"
-        iyz="-2.1253E-20"
-        izz="1.6012E-05" />
-    </inertial>
-    <visual>
-      <origin
-        xyz="0 0 0"
-        rpy="0 0 0" />
-      <geometry>
-        <mesh
-          filename="package://waiteronix/meshes/F_W_Front_Left.STL" />
-      </geometry>
-      <material
-        name="">
-        <color
-          rgba="0.50196 0.50196 1 1" />
-      </material>
-    </visual>
-    <collision>
-      <origin
-        xyz="0 0 0"
-        rpy="0 0 0" />
-      <geometry>
-        <mesh
-          filename="package://waiteronix/meshes/F_W_Front_Left.STL" />
-      </geometry>
-    </collision>
-  </link>
-  <joint
-    name="F_W_Front_Left_Joint"
-    type="fixed">
-    <origin
-      xyz="0 0 0"
-      rpy="0 0 0" />
-    <parent
-      link="base_link" />
-    <child
-      link="F_W_Front_Left" />
-    <axis
-      xyz="0 1 0" />
-  </joint>
-  <link
-    name="F_W_Front_Right">
-    <inertial>
-      <origin
-        xyz="0.13868 -0.123 2.4819E-14"
-        rpy="0 0 0" />
-      <mass
-        value="0.059636" />
-      <inertia
-        ixx="1.6012E-05"
-        ixy="5.4827E-21"
-        ixz="-3.2336E-22"
-        iyy="2.7287E-05"
-        iyz="-3.8765E-20"
-        izz="1.6012E-05" />
-    </inertial>
-    <visual>
-      <origin
-        xyz="0 0 0"
-        rpy="0 0 0" />
-      <geometry>
-        <mesh
-          filename="package://waiteronix/meshes/F_W_Front_Right.STL" />
-      </geometry>
-      <material
-        name="">
-        <color
-          rgba="0.50196 0.50196 1 1" />
-      </material>
-    </visual>
-    <collision>
-      <origin
-        xyz="0 0 0"
-        rpy="0 0 0" />
-      <geometry>
-        <mesh
-          filename="package://waiteronix/meshes/F_W_Front_Right.STL" />
-      </geometry>
-    </collision>
-  </link>
-  <joint
-    name="F_W_Front_Right_Joint"
-    type="fixed">
-    <origin
-      xyz="0 0 0"
-      rpy="0 0 0" />
-    <parent
-      link="base_link" />
-    <child
-      link="F_W_Front_Right" />
-    <axis
-      xyz="0 1 0" />
-  </joint>
-  <link
-    name="F_W_Back_Left">
-    <inertial>
-      <origin
-        xyz="-0.19 0.1215 -1.622E-14"
-        rpy="0 0 0" />
-      <mass
-        value="0.059636" />
-      <inertia
-        ixx="1.6012E-05"
-        ixy="2.3169E-21"
-        ixz="-1.6362E-21"
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