Commit message: adding voxel layer and modifying some parameters to config files and adding robot_footprint to urdf

File: waiteronix_description/urdf/waiteronix.xacro (robot description, xacro)
@@ -6,4 +6,6 @@
   name="waiteronix_description" xmlns:xacro="http://www.ros.org/wiki/xacro">
   <xacro:include filename="$(find waiteronix_description)/urdf/waiteronix.gazebo"/>
+  <link name="robot_footprint">
+  </link>
   <link
     name="base_link">
@@ -86,4 +88,8 @@
     </collision>
   </link>
+      <joint name="dummy_joint" type="fixed">
+    <parent link="robot_footprint"/>
+    <child link="base_link"/>
+   </joint>
   <joint
     name="right_wheel_joint"
